File: GOAT/Max_MainPCB/Max_MainPCB.kicad_sch (KiCad schematic)
At the start: 33 parts, among them IC1 INA228AQDGSRQ1, IC2 AP63205WU-7, J10 Screw_Terminal_01x02, J11 Screw_Terminal_01x03, J12 Screw_Terminal_01x02, J13 Screw_Terminal_01x03, J14 Screw_Terminal_01x02, J15 Screw_Terminal_01x02, J16 Screw_Terminal_01x03, J17 Screw_Terminal_01x03, J4 Screw_Terminal_01x02, J5 Screw_Terminal_01x02, J6 Screw_Terminal_01x04, J8 Screw_Terminal_01x02, J9 Screw_Terminal_01x03, U1 SEEEDUINO XIAO ESP32-C3

Commit message: update
Other:
- note removed: "Check all R,L,C sizes"
- note removed: "Check connections on 8-9-10"
Changed lines of the file:
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@@
     (effects (font (size 1.27 1.27)) (justify left bottom))
-  )
-  (text "Check connections on 8-9-10" (at 290.83 30.48 0)
-    (effects (font (size 3 3) (thickness 1) bold (color 255 30 28 1)) (justify left bottom))
   )
   (text "DC-DC Buck converter" (at 49.53 72.39 0)
     (effects (font (size 3 3) (thickness 1) bold) (justify left bottom))
   )
-  (text "Check all R,L,C sizes" (at 90.17 7.62 0)
-    (effects (font (size 3 3) (thickness 1) bold (color 255 30 28 1)) (justify left bottom))
-  )
   (text "Motor 1" (at 27.94 151.13 0)
